Commit message: [UPDATE] correccion angulos en el lidar simulado

File: car_description/robot/car.urdf.xacro (robot description, xacro)
@@ -1,41 +1,41 @@
 <?xml version="1.0"?>
 <robot xmlns:xacro="http://ros.org/wiki/xacro" name="car">
-  <xacro:arg name="wheel_diameter" default="0.112"/>
-  <xacro:property name="wheel_radius" value="${$(arg wheel_diameter)/2}"/>
-  <xacro:property name="wheel_width" value="0.047"/>
-  <xacro:property name="wheel_friction" value="0.8"/>
-  <xacro:property name="wheelbase_length" value="0.3429"/>
-  <xacro:property name="front_wheelbase_width" value="0.25"/>
-  <xacro:property name="rear_wheelbase_width" value="0.25"/>
-  <xacro:property name="wheel_mass" value="0.1"/>
-  <xacro:property name="total_mass" value = "3.0"/>
-  <xacro:property name="shock_travel" value = "0.09"/>
-  <xacro:property name="chassis_height" value = "0.06"/>
-  <xacro:property name="chassis_elevation" value = "-0.01"/>
-  <xacro:property name="chassis_mass" value = "${total_mass-4*wheel_mass}"/>
+  <xacro:arg name="wheel_diameter" default="0.112" />
+  <xacro:property name="wheel_radius" value="${$(arg wheel_diameter)/2}" />
+  <xacro:property name="wheel_width" value="0.047" />
+  <xacro:property name="wheel_friction" value="0.8" />
+  <xacro:property name="wheelbase_length" value="0.3429" />
+  <xacro:property name="front_wheelbase_width" value="0.25" />
+  <xacro:property name="rear_wheelbase_width" value="0.25" />
+  <xacro:property name="wheel_mass" value="0.1" />
+  <xacro:property name="total_mass" value="3.0" />
+  <xacro:property name="shock_travel" value="0.09" />
+  <xacro:property name="chassis_height" value="0.06" />
+  <xacro:property name="chassis_elevation" value="-0.01" />
+  <xacro:property name="chassis_mass" value="${total_mass-4*wheel_mass}" />
   <xacro:macro name="cylinder_inertia" params="m r h">
-        <inertia  ixx="${m*(3*r*r+h*h)/12}" ixy = "0" ixz = "0"
-                    iyy="${m*(3*r*r+h*h)/12}" iyz = "0"
-                    izz="${m*r*r/2}" />
+    <inertia ixx="${m*(3*r*r+h*h)/12}" ixy="0" ixz="0"
+      iyy="${m*(3*r*r+h*h)/12}" iyz="0"
+      izz="${m*r*r/2}" />
   </xacro:macro>
   <xacro:macro name="box_inertia" params="m x y z">
-          <inertia  ixx="${m*(y*y+z*z)/12}" ixy = "0" ixz = "0"
-                    iyy="${m*(x*x+z*z)/12}" iyz = "0"
-                    izz="${m*(x*x+z*z)/12}" />
+    <inertia ixx="${m*(y*y+z*z)/12}" ixy="0" ixz="0"
+      iyy="${m*(x*x+z*z)/12}" iyz="0"
+      izz="${m*(x*x+z*z)/12}" />
   </xacro:macro>
   <xacro:macro name="sphere_inertia" params="m r">
-          <inertia  ixx="${2*m*r*r/5}" ixy = "0" ixz = "0"
-                    iyy="${2*m*r*r/5}" iyz = "0"
-                    izz="${2*m*r*r/5}" />
+    <inertia ixx="${2*m*r*r/5}" ixy="0" ixz="0"
+      iyy="${2*m*r*r/5}" iyz="0"
+      izz="${2*m*r*r/5}" />
   </xacro:macro>
   <xacro:macro name="cylinder_inertial" params="m r h">
     <inertial>
-      <mass value="${m}"/>
-      <xacro:cylinder_inertia m="${m}" r="${r}" h="${h}"/>
+      <mass value="${m}" />
+      <xacro:cylinder_inertia m="${m}" r="${r}" h="${h}" />
     </inertial>
   </xacro:macro>
-  <link name="base_footprint"/>
-  <link name="base_link"/>
-<!--
+  <link name="base_footprint" />
+  <link name="base_link" />
+  <!--
   <link name="base_link">
     <visual>
@@ -64,15 +64,16 @@
     <visual>
       <geometry>
-        <box size="${wheelbase_length} ${front_wheelbase_width} ${chassis_height}"/>
-      </geometry>
-    </visual>
-    <collision>
-      <geometry>
-        <box size="${wheelbase_length} ${front_wheelbase_width} ${chassis_height}"/>
-      </geometry>
-    </collision>
-    <inertial>
-      <mass value="${chassis_mass}"/>
-      <xacro:box_inertia m="${chassis_mass}" x="${wheelbase_length}" y="${front_wheelbase_width}" z="${chassis_height}"/>
+        <box size="${wheelbase_length} ${front_wheelbase_width} ${chassis_height}" />
+      </geometry>
+    </visual>
+    <collision>
+      <geometry>
+        <box size="${wheelbase_length} ${front_wheelbase_width} ${chassis_height}" />
+      </geometry>
+    </collision>
+    <inertial>
+      <mass value="${chassis_mass}" />
+      <xacro:box_inertia m="${chassis_mass}" x="${wheelbase_length}" y="${front_wheelbase_width}"
+        z="${chassis_height}" />
     </inertial>
   </link>
@@ -80,56 +81,58 @@
     <visual>
       <geometry>
-        <cylinder length="${wheel_width}" radius="${wheel_radius}"/>
-      </geometry>
-      <material name="black">
-        <color rgba="0 0 0 1"/>
-      </material>
-    </visual>
-    <collision>
-      <geometry>
-        <cylinder length="${wheel_width}" radius="${wheel_radius}"/>
-      </geometry>
-    </collision>
-    <xacro:cylinder_inertial m="${wheel_mass}" r="${wheel_radius}" h="${wheel_width}"/>
+        <cylinder length="${wheel_width}" radius="${wheel_radius}" />
+      </geometry>
+      <material name="black">
+        <color rgba="0 0 0 1" />
+      </material>
+    </visual>
+    <collision>
+      <geometry>
+        <cylinder length="${wheel_width}" radius="${wheel_radius}" />
+      </geometry>
+    </collision>
+    <xacro:cylinder_inertial m="${wheel_mass}" r="${wheel_radius}" h="${wheel_width}" />
   </link>
   <link name="laser_scanner_link">
     <collision>
-      <origin xyz="0 0 0" rpy="0 0 0"/>
-      <geometry>
-        <box size=".127 0.1016 0.0508"/>
-      </geometry>
-    </collision>
-    <visual>
-      <origin xyz="0 0 0" rpy="0 0 0"/>
-      <geometry>
-        <box size=".127 0.1016 0.0508"/>
-      </geometry>
-    </visual>
-    <inertial>
-      <mass value="1e-5"/>
-      <origin xyz="0 0 0" rpy="0 0 0"/>
-      <inertia ixx="1e-6" ixy="0" ixz="0" iyy="1e-6" iyz="0" izz="1e-6"/>
+      <origin xyz="0 0 0" rpy="0 0 0" />
+      <geometry>
+        <box size=".127 0.1016 0.0508" />
+      </geometry>
+    </collision>
+    <visual>
+      <origin xyz="0 0 0" rpy="0 0 0" />
+      <geometry>
+        <box size=".127 0.1016 0.0508" />
+      </geometry>
+    </visual>
+    <inertial>
+      <mass value="1e-5" />
+      <origin xyz="0 0 0" rpy="0 0 0" />
+      <inertia ixx="1e-6" ixy="0" ixz="0" iyy="1e-6" iyz="0" izz="1e-6" />
     </inertial>
   </link>
   <gazebo reference="laser_scanner_link">
     <sensor type="ray" name="laser_scanner">
-    <always_on>true</always_on>
-    <!-- <visualize>true</visualize> -->
-    <update_rate>3</update_rate>
-    <ray>
-      <scan>
-        <horizontal>
-          <samples>360</samples>
-          <resolution>1</resolution>
-          <min_angle>${-pi}</min_angle>
-          <max_angle>${pi}</max_angle>
-        </horizontal>
-      </scan>
-      <range>
-        <min>0.30</min>
-        <max>25.0</max>
-        <resolution>0.1</resolution>
-      </range>
-    </ray>
+      <always_on>true</always_on>
+      <!-- <visualize>true</visualize> -->
+      <update_rate>3</update_rate>
+      <ray>
+        <scan>
+          <horizontal>
+            <samples>360</samples>
+            <resolution>1</resolution>
+            <!-- <min_angle>${-pi}</min_angle>
+            <max_angle>${pi}</max_angle> -->
+            <min_angle>${0}</min_angle>
+            <max_angle>${2*pi}</max_angle>
+          </horizontal>
+        </scan>
+        <range>
+          <min>0.1</min>
+          <max>25.0</max>
+          <resolution>0.1</resolution>
+        </range>
+      </ray>
       <plugin name="scan" filename="libgazebo_ros_ray_sensor.so">
         <ros>
@@ -144,71 +147,71 @@
     <visual>
       <geometry>
-        <cylinder length="${wheel_width}" radius="${wheel_radius}"/>
-      </geometry>
-      <material name="black">
-        <color rgba="0 0 0 1"/>
-      </material>
-    </visual>
-    <collision>
-      <geometry>
-        <cylinder length="${wheel_width}" radius="${wheel_radius}"/>
-      </geometry>
-    </collision>
-    <xacro:cylinder_inertial m="${wheel_mass}" r="${wheel_radius}" h="${wheel_width}"/>
+        <cylinder length="${wheel_width}" radius="${wheel_radius}" />
+      </geometry>
+      <material name="black">
+        <color rgba="0 0 0 1" />
+      </material>
+    </visual>
+    <collision>
+      <geometry>
+        <cylinder length="${wheel_width}" radius="${wheel_radius}" />
+      </geometry>
+    </collision>
+    <xacro:cylinder_inertial m="${wheel_mass}" r="${wheel_radius}" h="${wheel_width}" />
   </link>
   <link name="front_left_wheel_steer">
     <visual>
       <geometry>
-        <cylinder length="0.01" radius="0.01"/>
-      </geometry>
-      <material name="black">
-        <color rgba="0 0 0 1"/>
-      </material>
-    </visual>
-    <collision>
-      <geometry>
-        <cylinder length="0.01" radius="0.01"/>
-      </geometry>
-    </collision>
-    <inertial>
-      <mass value="0.1"/>
+        <cylinder length="0.01" radius="0.01" />
+      </geometry>
+      <material name="black">
+        <color rgba="0 0 0 1" />
+      </material>
+    </visual>
+    <collision>
+      <geometry>
+        <cylinder length="0.01" radius="0.01" />
+      </geometry>
+    </collision>
+    <inertial>
+      <mass value="0.1" />
       <inertia ixx="5.1458e-5" iyy="5.1458e-5" izz="6.125e-5"
-               ixy="0" ixz="0" iyz="0"/>
-    </inertial>
-  </link>
-    <link name="front_left_wheel">
-    <visual>
-      <geometry>
-        <cylinder length="${wheel_width}" radius="${wheel_radius}"/>
-      </geometry>
-      <material name="black">
-        <color rgba="0 0 0 1"/>
-      </material>
-    </visual>
-    <collision>
-      <geometry>
-        <cylinder length="${wheel_width}" radius="${wheel_radius}"/>
-      </geometry>
-    </collision>
-    <xacro:cylinder_inertial m="${wheel_mass}" r="${wheel_radius}" h="${wheel_width}"/>
+        ixy="0" ixz="0" iyz="0" />
+    </inertial>
+  </link>
+  <link name="front_left_wheel">
+    <visual>
+      <geometry>
+        <cylinder length="${wheel_width}" radius="${wheel_radius}" />
+      </geometry>
+      <material name="black">
+        <color rgba="0 0 0 1" />
+      </material>
+    </visual>
+    <collision>
+      <geometry>
+        <cylinder length="${wheel_width}" radius="${wheel_radius}" />
+      </geometry>
+    </collision>
+    <xacro:cylinder_inertial m="${wheel_mass}" r="${wheel_radius}" h="${wheel_width}" />
   </link>
   <link name="front_right_wheel_steer">
     <visual>
       <geometry>
-        <cylinder length="0.01" radius="0.01"/>
-      </geometry>
-      <material name="black">
-        <color rgba="0 0 0 1"/>
-      </material>
-    </visual>
-    <collision>
-      <geometry>
-        <cylinder length="0.01" radius="0.01"/>
-      </geometry>
-    </collision>
-    <inertial>
-      <mass value="0.1"/>
+        <cylinder length="0.01" radius="0.01" />
+      </geometry>
+      <material name="black">
+        <color rgba="0 0 0 1" />
+      </material>
+    </visual>
+    <collision>
+      <geometry>
+        <cylinder length="0.01" radius="0.01" />
+      </geometry>
+    </collision>
+    <inertial>
+      <mass value="0.1" />
       <inertia ixx="5.1458e-5" iyy="5.1458e-5" izz="6.125e-5"
-               ixy="0" ixz="0" iyz="0"/>
+        ixy="0" ixz="0" iyz="0" />
     </inertial>
   </link>
@@ -216,187 +219,187 @@
     <visual>
       <geometry>
-        <cylinder length="${wheel_width}" radius="${wheel_radius}"/>
-      </geometry>
-      <material name="black">
-        <color rgba="0 0 0 1"/>
-      </material>
-    </visual>
-    <collision>
-      <geometry>
-        <cylinder length="${wheel_width}" radius="${wheel_radius}"/>
-      </geometry>
-    </collision>
-    <xacro:cylinder_inertial m="${wheel_mass}" r="${wheel_radius}" h="${wheel_width}"/>
+        <cylinder length="${wheel_width}" radius="${wheel_radius}" />
+      </geometry>
+      <material name="black">
+        <color rgba="0 0 0 1" />
+      </material>
+    </visual>
+    <collision>
+      <geometry>
+        <cylinder length="${wheel_width}" radius="${wheel_radius}" />
+      </geometry>
+    </collision>
+    <xacro:cylinder_inertial m="${wheel_mass}" r="${wheel_radius}" h="${wheel_width}" />
   </link>
   <link name="back_left_wheel_shock">
-      <visual>
-      <origin xyz="0 0 0.1" rpy="0 0 0"/>
-      <geometry>
-        <cylinder length="0.05" radius="0.01"/>
+    <visual>
+      <origin xyz="0 0 0.1" rpy="0 0 0" />
+      <geometry>
+        <cylinder length="0.05" radius="0.01" />
       </geometry>
       <material name="silver">
-        <color rgba="0.75 0.75 0.75 1"/>
-      </material>
-    </visual>
-    <collision>
-      <origin xyz="0 0 0.1" rpy="0 0 0"/>
-      <geometry>
-        <cylinder length="0.05" radius="0.01"/>
-      </geometry>
-    </collision>
-    <inertial>
-      <mass value="0.01"/>
+        <color rgba="0.75 0.75 0.75 1" />
+      </material>
+    </visual>
+    <collision>
+      <origin xyz="0 0 0.1" rpy="0 0 0" />
+      <geometry>
+        <cylinder length="0.05" radius="0.01" />
+      </geometry>
+    </collision>
+    <inertial>
+      <mass value="0.01" />
       <inertia ixx="0.015" iyy="0.0375" izz="0.0375"
-               ixy="0" ixz="0" iyz="0"/>
+        ixy="0" ixz="0" iyz="0" />
     </inertial>
   </link>
   <link name="back_right_wheel_shock">
     <visual>
-    <origin xyz="0 0 0.1" rpy="0 0 0"/>
-    <geometry>
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